File: UniBoard.kicad_pcb (KiCad board)
At the start: 2 copper layers, 1 part, among them J1 UniSat_BUS_40

Commit message: updated the base project stuff
Other:
- board outline added: 89 x 93.3 mm
Changed lines of the file:
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@@
-(kicad_pcb (version 20171130) (host pcbnew "(5.1.10)-1")
+(kicad_pcb (version 20171130) (host pcbnew "(5.1.10-1-10_14)")
   (general
     (thickness 1.6)
-    (drawings 0)
+    (drawings 4)
     (tracks 0)
     (zones 0)
@@
     (uvia_dia 0.3)
     (uvia_drill 0.1)
-    (add_net "Net-(J1-Pad1)")
-    (add_net "Net-(J1-Pad10)")
-    (add_net "Net-(J1-Pad11)")
-    (add_net "Net-(J1-Pad12)")
-    (add_net "Net-(J1-Pad13)")
-    (add_net "Net-(J1-Pad14)")
-    (add_net "Net-(J1-Pad15)")
-    (add_net "Net-(J1-Pad16)")
-    (add_net "Net-(J1-Pad17)")
-    (add_net "Net-(J1-Pad18)")
-    (add_net "Net-(J1-Pad19)")
-    (add_net "Net-(J1-Pad2)")
-    (add_net "Net-(J1-Pad20)")
-    (add_net "Net-(J1-Pad21)")
-    (add_net "Net-(J1-Pad22)")
-    (add_net "Net-(J1-Pad23)")
-    (add_net "Net-(J1-Pad24)")
-    (add_net "Net-(J1-Pad25)")
-    (add_net "Net-(J1-Pad26)")
-    (add_net "Net-(J1-Pad27)")
-    (add_net "Net-(J1-Pad28)")
-    (add_net "Net-(J1-Pad29)")
-    (add_net "Net-(J1-Pad3)")
-    (add_net "Net-(J1-Pad30)")
-    (add_net "Net-(J1-Pad31)")
-    (add_net "Net-(J1-Pad32)")
-    (add_net "Net-(J1-Pad33)")
-    (add_net "Net-(J1-Pad34)")
-    (add_net "Net-(J1-Pad35)")
-    (add_net "Net-(J1-Pad36)")
-    (add_net "Net-(J1-Pad37)")
-    (add_net "Net-(J1-Pad38)")
-    (add_net "Net-(J1-Pad39)")
-    (add_net "Net-(J1-Pad4)")
-    (add_net "Net-(J1-Pad40)")
-    (add_net "Net-(J1-Pad5)")
-    (add_net "Net-(J1-Pad6)")
-    (add_net "Net-(J1-Pad7)")
-    (add_net "Net-(J1-Pad8)")
-    (add_net "Net-(J1-Pad9)")
   )
   (module UniBoard:Bus40PinSocket_2x20_P2.54mm_Vertical (layer F.Cu)
@@
       (effects (font (size 1 1) (thickness 0.15)))
     )
+    (fp_line (start -2.54 -1.27) (end 0.27 -1.27) (layer F.Fab) (width 0.1))
+    (fp_line (start -3.81 0) (end -3.81 0) (layer F.Fab) (width 0.1))
+    (fp_line (start -3.81 0) (end -2.54 -1.27) (layer F.Fab) (width 0.1))
+    (fp_line (start 0.27 -1.27) (end 1.27 -1.27) (layer F.Fab) (width 0.1))
+    (fp_line (start 1.27 -1.27) (end 1.27 49.53) (layer F.Fab) (width 0.1))
+    (fp_line (start 1.27 49.53) (end -3.81 49.53) (layer F.Fab) (width 0.1))
+    (fp_line (start -3.81 49.53) (end -3.81 0) (layer F.Fab) (width 0.1))
+    (fp_line (start -3.87 -1.33) (end -1.27 -1.33) (layer F.SilkS) (width 0.12))
+    (fp_line (start -3.87 -1.33) (end -3.87 49.59) (layer F.SilkS) (width 0.12))
+    (fp_line (start -3.87 49.59) (end 1.33 49.59) (layer F.SilkS) (width 0.12))
+    (fp_line (start 1.33 1.27) (end 1.33 49.59) (layer F.SilkS) (width 0.12))
+    (fp_line (start -1.27 1.27) (end -3.81 1.27) (layer F.SilkS) (width 0.12))
+    (fp_line (start -1.27 -1.33) (end -1.27 1.27) (layer F.SilkS) (width 0.12))
+    (fp_line (start 1.33 -1.33) (end 1.33 1.27) (layer F.SilkS) (width 0.12))
+    (fp_line (start -1.27 -1.33) (end 1.33 -1.33) (layer F.SilkS) (width 0.12))
+    (fp_line (start -4.34 -1.8) (end 1.76 -1.8) (layer F.CrtYd) (width 0.05))
+    (fp_line (start 1.76 -1.8) (end 1.76 50) (layer F.CrtYd) (width 0.05))
+    (fp_line (start 1.76 50) (end -4.34 50) (layer F.CrtYd) (width 0.05))
+    (fp_line (start -4.34 50) (end -4.34 -1.8) (layer F.CrtYd) (width 0.05))
     (fp_text user %R (at -1.27 24.13 90) (layer F.Fab)
       (effects (font (size 1 1) (thickness 0.15)))
     )
-    (fp_line (start -4.34 50) (end -4.34 -1.8) (layer F.CrtYd) (width 0.05))
-    (fp_line (start 1.76 50) (end -4.34 50) (layer F.CrtYd) (width 0.05))
-    (fp_line (start 1.76 -1.8) (end 1.76 50) (layer F.CrtYd) (width 0.05))
-    (fp_line (start -4.34 -1.8) (end 1.76 -1.8) (layer F.CrtYd) (width 0.05))
-    (fp_line (start -1.27 -1.33) (end 1.33 -1.33) (layer F.SilkS) (width 0.12))
-    (fp_line (start 1.33 -1.33) (end 1.33 1.27) (layer F.SilkS) (width 0.12))
-    (fp_line (start -1.27 -1.33) (end -1.27 1.27) (layer F.SilkS) (width 0.12))
-    (fp_line (start -1.27 1.27) (end -3.81 1.27) (layer F.SilkS) (width 0.12))
-    (fp_line (start 1.33 1.27) (end 1.33 49.59) (layer F.SilkS) (width 0.12))
-    (fp_line (start -3.87 49.59) (end 1.33 49.59) (layer F.SilkS) (width 0.12))
-    (fp_line (start -3.87 -1.33) (end -3.87 49.59) (layer F.SilkS) (width 0.12))
-    (fp_line (start -3.87 -1.33) (end -1.27 -1.33) (layer F.SilkS) (width 0.12))
-    (fp_line (start -3.81 49.53) (end -3.81 0) (layer F.Fab) (width 0.1))
-    (fp_line (start 1.27 49.53) (end -3.81 49.53) (layer F.Fab) (width 0.1))
-    (fp_line (start 1.27 -1.27) (end 1.27 49.53) (layer F.Fab) (width 0.1))
-    (fp_line (start 0.27 -1.27) (end 1.27 -1.27) (layer F.Fab) (width 0.1))
-    (fp_line (start -3.81 0) (end -2.54 -1.27) (layer F.Fab) (width 0.1))
-    (fp_line (start -3.81 0) (end -3.81 0) (layer F.Fab) (width 0.1))
-    (fp_line (start -2.54 -1.27) (end 0.27 -1.27) (layer F.Fab) (width 0.1))
     (pad 39 thru_hole oval (at -2.54 48.26) (size 1.7 1.7) (drill 1) (layers *.Cu *.Mask))
     (pad 40 thru_hole oval (at 0 48.26) (size 1.7 1.7) (drill 1) (layers *.Cu *.Mask))
@@
     )
   )
+  (gr_line (start 188.49 133.3) (end 188.49 40) (layer Edge.Cuts) (width 0.05))
+  (gr_line (start 99.49 133.3) (end 99.49 40) (layer Edge.Cuts) (width 0.05))
+  (gr_line (start 99.49 133.3) (end 188.49 133.3) (layer Edge.Cuts) (width 0.05))
+  (gr_line (start 99.49 40) (end 188.49 40) (layer Edge.Cuts) (width 0.05))
 )

Commit message: bottom 2 are ok
Parts:
- added H1: 3.2, MountingHole:MountingHole_3.2mm_M3_Pad, F.Cu at (106.0, 43.5)
- added H2: 4, MountingHole:MountingHole_4mm, F.Cu at (113.3, 48.4)
- added H3: 3.2, MountingHole:MountingHole_3.2mm_M3_Pad, F.Cu at (182.0, 43.5)
- added H4: 4, MountingHole:MountingHole_4mm, F.Cu at (173.7, 48.3)
- added H5: 3.2, MountingHole:MountingHole_3.2mm_M3_Pad, F.Cu at (106.0, 129.8)
- added H6: 3.2, MountingHole:MountingHole_3.2mm_M3_Pad, F.Cu at (182.0, 129.8)
- moved J1 154.8 mm to (167.6, 49.7), turned to 270 degrees
Connections:
- J1 pad 1: (no net) -> Net-(J1-Pad1)
- J1 pad 10: (no net) -> Net-(J1-Pad10)
- J1 pad 11: (no net) -> Net-(J1-Pad11)
- J1 pad 12: (no net) -> Net-(J1-Pad12)
- J1 pad 13: (no net) -> Net-(J1-Pad13)
- J1 pad 14: (no net) -> Net-(J1-Pad14)
- J1 pad 15: (no net) -> Net-(J1-Pad15)
- J1 pad 16: (no net) -> Net-(J1-Pad16)
- J1 pad 17: (no net) -> Net-(J1-Pad17)
- J1 pad 18: (no net) -> Net-(J1-Pad18)
- J1 pad 19: (no net) -> Net-(J1-Pad19)
- J1 pad 2: (no net) -> Net-(J1-Pad2)
- J1 pad 20: (no net) -> Net-(J1-Pad20)
- J1 pad 21: (no net) -> Net-(J1-Pad21)
- J1 pad 22: (no net) -> Net-(J1-Pad22)
- J1 pad 23: (no net) -> Net-(J1-Pad23)
- J1 pad 24: (no net) -> Net-(J1-Pad24)
- J1 pad 25: (no net) -> Net-(J1-Pad25)
- J1 pad 26: (no net) -> Net-(J1-Pad26)
- J1 pad 27: (no net) -> Net-(J1-Pad27)
- J1 pad 28: (no net) -> Net-(J1-Pad28)
- J1 pad 29: (no net) -> Net-(J1-Pad29)
- J1 pad 3: (no net) -> Net-(J1-Pad3)
- J1 pad 30: (no net) -> Net-(J1-Pad30)
- J1 pad 31: (no net) -> Net-(J1-Pad31)
- J1 pad 32: (no net) -> Net-(J1-Pad32)
- J1 pad 33: (no net) -> Net-(J1-Pad33)
- J1 pad 34: (no net) -> Net-(J1-Pad34)
- J1 pad 35: (no net) -> Net-(J1-Pad35)
- J1 pad 36: (no net) -> Net-(J1-Pad36)
- J1 pad 37: (no net) -> Net-(J1-Pad37)
- J1 pad 38: (no net) -> Net-(J1-Pad38)
- J1 pad 39: (no net) -> Net-(J1-Pad39)
- J1 pad 4: (no net) -> Net-(J1-Pad4)
- J1 pad 40: (no net) -> Net-(J1-Pad40)
- J1 pad 5: (no net) -> Net-(J1-Pad5)
- J1 pad 6: (no net) -> Net-(J1-Pad6)
- J1 pad 7: (no net) -> Net-(J1-Pad7)
- J1 pad 8: (no net) -> Net-(J1-Pad8)
- J1 pad 9: (no net) -> Net-(J1-Pad9)
Other:
- outline, holes or cut-outs redrawn
