File: UniBoard.sch (KiCad schematic (older format))
At the start: 1 part, among them J1 UniSat_BUS_40

Commit message: bottom 2 are ok
Parts:
- added H1, H3, H5, H6: 3.2, MountingHole:MountingHole_3.2mm_M3_Pad, symbol Mechanical:MountingHole_Pad
- added H2, H4: 4, MountingHole:MountingHole_4mm, symbol Mechanical:MountingHole
Changed lines of the file:
@@
 	0    1    1    0
 $EndComp
+$Comp
+L Mechanical:MountingHole_Pad H1
+U 1 1 618CFB30
+P 8200 1000
+F 0 "H1" H 8300 1049 50  0000 L CNN
+F 1 "3.2" H 8300 958 50  0000 L CNN
+F 2 "MountingHole:MountingHole_3.2mm_M3_Pad" H 8200 1000 50  0001 C CNN
+F 3 "~" H 8200 1000 50  0001 C CNN
+	1    8200 1000
+	1    0    0    -1
+$EndComp
+$Comp
+L Mechanical:MountingHole H2
+U 1 1 618D0D67
+P 8200 1300
+F 0 "H2" H 8300 1346 50  0000 L CNN
+F 1 "4" H 8300 1255 50  0000 L CNN
+F 2 "MountingHole:MountingHole_4mm" H 8200 1300 50  0001 C CNN
+F 3 "~" H 8200 1300 50  0001 C CNN
+	1    8200 1300
+	1    0    0    -1
+$EndComp
+$Comp
+L Mechanical:MountingHole_Pad H3
+U 1 1 618D115B
+P 8550 1000
+F 0 "H3" H 8650 1049 50  0000 L CNN
+F 1 "3.2" H 8650 958 50  0000 L CNN
+F 2 "MountingHole:MountingHole_3.2mm_M3_Pad" H 8550 1000 50  0001 C CNN
+F 3 "~" H 8550 1000 50  0001 C CNN
+	1    8550 1000
+	1    0    0    -1
+$EndComp
+$Comp
+L Mechanical:MountingHole_Pad H5
+U 1 1 618D1327
+P 8900 1000
+F 0 "H5" H 9000 1049 50  0000 L CNN
+F 1 "3.2" H 9000 958 50  0000 L CNN
+F 2 "MountingHole:MountingHole_3.2mm_M3_Pad" H 8900 1000 50  0001 C CNN
+F 3 "~" H 8900 1000 50  0001 C CNN
+	1    8900 1000
+	1    0    0    -1
+$EndComp
+$Comp
+L Mechanical:MountingHole_Pad H6
+U 1 1 618D1620
+P 9250 1000
+F 0 "H6" H 9350 1049 50  0000 L CNN
+F 1 "3.2" H 9350 958 50  0000 L CNN
+F 2 "MountingHole:MountingHole_3.2mm_M3_Pad" H 9250 1000 50  0001 C CNN
+F 3 "~" H 9250 1000 50  0001 C CNN
+	1    9250 1000
+	1    0    0    -1
+$EndComp
+$Comp
+L Mechanical:MountingHole H4
+U 1 1 618D1889
+P 8550 1300
+F 0 "H4" H 8650 1346 50  0000 L CNN
+F 1 "4" H 8650 1255 50  0000 L CNN
+F 2 "MountingHole:MountingHole_4mm" H 8550 1300 50  0001 C CNN
+F 3 "~" H 8550 1300 50  0001 C CNN
+	1    8550 1300
+	1    0    0    -1
+$EndComp
 $EndSCHEMATC

Commit message: added silk screen
Other:
- note added: "Essential Parts"
- note added: "UniSat Bus (40PIN)"
- moved on the sheet: H1, H2, H3, H4, H5, H6, J1
Changed lines of the file:
@@
 encoding utf-8
 Sheet 1 1
-Title ""
-Date ""
-Rev ""
-Comp ""
+Title "UniSat UniBoard Base"
+Date "2021-11-11"
+Rev "v1.0"
+Comp "UniSat Nano-satellite Educational Programme for Girls"
 Comment1 ""
 Comment2 ""
-Comment3 ""
-Comment4 ""
+Comment3 "2021 Almaty "
+Comment4 "by Yaakov Azat (@azataiot)"
 $EndDescr
-$Comp
-L UniBoard:UniSat_BUS_40 J1
-U 1 1 618C35C1
-P 2650 1400
-F 0 "J1" V 2559 1488 50  0000 L CNN
-F 1 "UniSat_BUS_40" V 2650 1488 50  0000 L CNN
-F 2 "UniBoard:Bus40PinSocket_2x20_P2.54mm_Vertical" V 2650 1600 50  0001 C CNN
-F 3 "https://docs.google.com/spreadsheets/d/1PAcDkhzehB7XnIJytJIB0ZRkse9mW8csUumpt_BZlxQ/edit?usp=sharing" V 2741 1488 50  0000 L CNN
-	1    2650 1400
-	0    1    1    0
-$EndComp
 $Comp
 L Mechanical:MountingHole_Pad H1
 U 1 1 618CFB30
-P 8200 1000
-F 0 "H1" H 8300 1049 50  0000 L CNN
-F 1 "3.2" H 8300 958 50  0000 L CNN
-F 2 "MountingHole:MountingHole_3.2mm_M3_Pad" H 8200 1000 50  0001 C CNN
-F 3 "~" H 8200 1000 50  0001 C CNN
-	1    8200 1000
+P 3550 1150
+F 0 "H1" H 3650 1199 50  0000 L CNN
+F 1 "3.2" H 3650 1108 50  0000 L CNN
+F 2 "MountingHole:MountingHole_3.2mm_M3_Pad" H 3550 1150 50  0001 C CNN
+F 3 "~" H 3550 1150 50  0001 C CNN
+	1    3550 1150
 	1    0    0    -1
 $EndComp
@@
 L Mechanical:MountingHole H2
 U 1 1 618D0D67
-P 8200 1300
-F 0 "H2" H 8300 1346 50  0000 L CNN
-F 1 "4" H 8300 1255 50  0000 L CNN
-F 2 "MountingHole:MountingHole_4mm" H 8200 1300 50  0001 C CNN
-F 3 "~" H 8200 1300 50  0001 C CNN
-	1    8200 1300
+P 3550 1450
+F 0 "H2" H 3650 1496 50  0000 L CNN
+F 1 "4" H 3650 1405 50  0000 L CNN
+F 2 "MountingHole:MountingHole_4mm" H 3550 1450 50  0001 C CNN
+F 3 "~" H 3550 1450 50  0001 C CNN
+	1    3550 1450
 	1    0    0    -1
 $EndComp
@@
 L Mechanical:MountingHole_Pad H3
 U 1 1 618D115B
-P 8550 1000
-F 0 "H3" H 8650 1049 50  0000 L CNN
-F 1 "3.2" H 8650 958 50  0000 L CNN
-F 2 "MountingHole:MountingHole_3.2mm_M3_Pad" H 8550 1000 50  0001 C CNN
-F 3 "~" H 8550 1000 50  0001 C CNN
-	1    8550 1000
+P 3900 1150
+F 0 "H3" H 4000 1199 50  0000 L CNN
+F 1 "3.2" H 4000 1108 50  0000 L CNN
+F 2 "MountingHole:MountingHole_3.2mm_M3_Pad" H 3900 1150 50  0001 C CNN
+F 3 "~" H 3900 1150 50  0001 C CNN
+	1    3900 1150
 	1    0    0    -1
 $EndComp
@@
 L Mechanical:MountingHole_Pad H5
 U 1 1 618D1327
-P 8900 1000
-F 0 "H5" H 9000 1049 50  0000 L CNN
-F 1 "3.2" H 9000 958 50  0000 L CNN
-F 2 "MountingHole:MountingHole_3.2mm_M3_Pad" H 8900 1000 50  0001 C CNN
-F 3 "~" H 8900 1000 50  0001 C CNN
-	1    8900 1000
+P 4250 1150
+F 0 "H5" H 4350 1199 50  0000 L CNN
+F 1 "3.2" H 4350 1108 50  0000 L CNN
+F 2 "MountingHole:MountingHole_3.2mm_M3_Pad" H 4250 1150 50  0001 C CNN
+F 3 "~" H 4250 1150 50  0001 C CNN
+	1    4250 1150
 	1    0    0    -1
 $EndComp
@@
 L Mechanical:MountingHole_Pad H6
 U 1 1 618D1620
-P 9250 1000
-F 0 "H6" H 9350 1049 50  0000 L CNN
-F 1 "3.2" H 9350 958 50  0000 L CNN
-F 2 "MountingHole:MountingHole_3.2mm_M3_Pad" H 9250 1000 50  0001 C CNN
-F 3 "~" H 9250 1000 50  0001 C CNN
-	1    9250 1000
+P 4600 1150
+F 0 "H6" H 4700 1199 50  0000 L CNN
+F 1 "3.2" H 4700 1108 50  0000 L CNN
+F 2 "MountingHole:MountingHole_3.2mm_M3_Pad" H 4600 1150 50  0001 C CNN
+F 3 "~" H 4600 1150 50  0001 C CNN
+	1    4600 1150
 	1    0    0    -1
 $EndComp
@@
 L Mechanical:MountingHole H4
 U 1 1 618D1889
-P 8550 1300
-F 0 "H4" H 8650 1346 50  0000 L CNN
-F 1 "4" H 8650 1255 50  0000 L CNN
-F 2 "MountingHole:MountingHole_4mm" H 8550 1300 50  0001 C CNN
-F 3 "~" H 8550 1300 50  0001 C CNN
-	1    8550 1300
+P 3900 1450
+F 0 "H4" H 4000 1496 50  0000 L CNN
+F 1 "4" H 4000 1405 50  0000 L CNN
+F 2 "MountingHole:MountingHole_4mm" H 3900 1450 50  0001 C CNN
+F 3 "~" H 3900 1450 50  0001 C CNN
+	1    3900 1450
 	1    0    0    -1
 $EndComp
+$Comp
+L UniBoard:UniSat_BUS_40 J1
+U 1 1 618C35C1
+P 2750 1500
+F 0 "J1" V 2400 1600 50  0000 L CNN
+F 1 "UniSat_BUS_40" H 2600 1650 50  0000 L CNN
+F 2 "UniBoard:Bus40PinSocket_2x20_P2.54mm_Vertical" V 2750 1700 50  0001 C CNN
+F 3 "https://docs.google.com/spreadsheets/d/1PAcDkhzehB7XnIJytJIB0ZRkse9mW8csUumpt_BZlxQ/edit?usp=sharing" V 2841 1588 50  0001 L CNN
+	1    2750 1500
+	0    1    1    0
+$EndComp
+Wire Notes Line
+	3100 750  3100 2300
+Wire Notes Line
+	3100 2300 650  2300
+Wire Notes Line
+	650  2300 650  750
+Wire Notes Line
+	650  750  3100 750
+Text Notes 650  700  0    50   ~ 0
+UniSat Bus (40PIN)
+Wire Notes Line
+	5100 750  5100 2300
+Wire Notes Line
+	5100 2300 3350 2300
+Wire Notes Line
+	3350 2300 3350 750
+Wire Notes Line
+	3350 750  5100 750
+Text Notes 3350 700  0    50   ~ 0
+Essential Parts
 $EndSCHEMATC
